File: powersource.kicad_sch (KiCad schematic)
At the start: 110 parts, among them T1 Transformer_1P_SS

Commit message: Upgrade
Connections:
- net +12v: now also L8.4; no longer L8.2
- net -12v: now also L8.2; no longer L8.4
Changed lines of the file:
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@@
 		)
 	)
-	(global_label "+12v"
+	(global_label "-12v"
 		(shape input)
 		(at 247.65 81.28 0)
@@
 		)
 	)
-	(global_label "-12v"
+	(global_label "+12v"
 		(shape input)
 		(at 242.57 76.2 0)

Commit message: Upgrade
Connections:
- net +12v PWM: no longer C19.1
- net at T1.1 (AA): now also C19.1
Other:
- note added: "But this is not a solution of my problems criminals just continue to use and controll me from power sources with transformers or coils maybe I use transformerless in future"
- note added: "Line"
Changed lines of the file:
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@@
-	)
-	(junction
-		(at 114.3 87.63)
-		(diameter 0)
-		(color 0 0 0 0)
 	)
 	(junction
@@
 	(wire
 		(pts
+			(xy 114.3 97.79) (xy 99.06 97.79)
+		)
+		(stroke
+			(width 0)
+			(type default)
+		)
+	)
+	(wire
+		(pts
 			(xy 64.77 82.55) (xy 54.61 82.55)
 		)
@@
 	(wire
 		(pts
-			(xy 93.98 87.63) (xy 114.3 87.63)
-		)
-		(stroke
-			(width 0)
-			(type default)
-		)
-	)
-	(wire
-		(pts
 			(xy 182.88 86.36) (xy 182.88 90.17)
 		)
@@
 	(wire
 		(pts
+			(xy 67.31 102.87) (xy 67.31 91.44)
+		)
+		(stroke
+			(width 0)
+			(type default)
+		)
+	)
+	(wire
+		(pts
 			(xy 162.56 72.39) (xy 162.56 86.36)
 		)
@@
 	(wire
 		(pts
-			(xy 114.3 87.63) (xy 116.84 87.63)
+			(xy 93.98 87.63) (xy 116.84 87.63)
 		)
 		(stroke
@@
 	(wire
 		(pts
+			(xy 99.06 97.79) (xy 99.06 102.87)
+		)
+		(stroke
+			(width 0)
+			(type default)
+		)
+	)
+	(wire
+		(pts
 			(xy 120.65 109.22) (xy 130.81 109.22)
 		)
@@
 	(wire
 		(pts
+			(xy 99.06 102.87) (xy 67.31 102.87)
+		)
+		(stroke
+			(width 0)
+			(type default)
+		)
+	)
+	(wire
+		(pts
 			(xy 138.43 95.25) (xy 147.32 95.25)
 		)
@@
 	(wire
 		(pts
-			(xy 114.3 87.63) (xy 114.3 97.79)
-		)
-		(stroke
-			(width 0)
-			(type default)
-		)
-	)
-	(wire
-		(pts
 			(xy 167.64 138.43) (xy 167.64 149.86)
 		)
@@
 		(pts
 			(xy 93.98 91.44) (xy 93.98 87.63)
+		)
+		(stroke
+			(width 0)
+			(type default)
+		)
+	)
+	(wire
+		(pts
+			(xy 67.31 91.44) (xy 72.39 91.44)
 		)
 		(stroke
@@
 		(fill
 			(type none)
+		)
+	)
+	(text "Line\n"
+		(exclude_from_sim no)
+		(at 69.596 90.17 0)
+		(effects
+			(font
+				(size 1.27 1.27)
+			)
 		)
 	)
@@
 		(effects
 			(font
+				(size 1.27 1.27)
+			)
+		)
+	)
+	(text "But this is not a solution of my problems\ncriminals just continue to use and controll me from \npower sources with transformers or coils\nmaybe I use transformerless in future"
+		(exclude_from_sim no)
+		(at 82.296 111.252 0)
+		(effects
+			(font

Commit message: Upgrade
Parts:
- removed C19: C, symbol Device:C
- removed D1: D, symbol Device:D
- removed L6, L7: L, symbol Device:L
- removed L8: 2-3 turns, symbol Device:L_Ferrite_Coupled_Small
- removed T1: Transformer_1P_SS, symbol Device:Transformer_1P_SS
- added C100: 33nF, symbol Device:C
- added C101: 100mkF, symbol Device:C_Polarized
- added C102, C112, C83, C92: 10nF, symbol Device:C
- added C103: 10mkF, symbol Device:C_Polarized
- added C104, C113, C79, C93: 2.2mkF, symbol Device:C_Polarized
- added C105: 2.2nF, symbol Device:C
- added C106: 33mkF, symbol Device:C_Polarized
- added C107: 680pF, symbol Device:C
- added C108: 330mkF, symbol Device:C_Polarized
- added C109: 22000mkF, symbol Device:C_Polarized
- added C110: 22nF, symbol Device:C
- added C111, C78, C91: 220mkF, symbol Device:C_Polarized
- added C19, C98: 470mkF, symbol Device:C_Polarized
- added C75, C99: 1000mkF, symbol Device:C_Polarized
- added C76, C96: 47mkF, symbol Device:C_Polarized
- added C77, C94: 4.7mkF, symbol Device:C_Polarized
- added C80: 15nF, symbol Device:C
- added C81: 800pF, symbol Device:C
- added C82: 221pF, symbol Device:C
- added C84: 6.8mkF, symbol Device:C_Polarized
- added C85: 100nF, symbol Device:C
- added C86: 68mkF, symbol Device:C_Polarized
- added C87: 470pF, symbol Device:C
- added C88: 680mkF, symbol Device:C_Polarized
- added C89: 2200mkF, symbol Device:C_Polarized
- added C90: 4.7nF, symbol Device:C
- added C95: 1nF, symbol Device:C
- added C97: 3.3pF, symbol Device:C
- added L6: 60 turns, symbol Device:L_Coupled
- added S1, S2, S3, S4: S-changeover, symbol PCM_Elektuur:S-changeover
Connections:
- net +12v: now also C59.1, C60.1, C61.1, C62.1, C63.1, C64.1, C71.2, C72.2, C73.2, C74.2, L1.4
- net Ground: now reaches C65.2, C66.2, C67.2, C68.2, C69.2, C70.2, C71.1, C72.1, C73.1, C74.1, L1.2
- net FH3: now reaches C21.2, C23.2, C25.2, C27.2, C28.1, C29.1, C30.1, C31.1, C32.1, C34.2, C40.2, C41.2, C42.2, C43.2, C44.2, C46.2, L2.4
- net FH3: now also L6.2, S2.1
- net FH1: now reaches C13.1, C14.1, C15.1, C16.1, C17.1, L4.1, L5.2
- net FH1: now also S1.1
- net FH2: now reaches C1.1, C2.1, C3.1, C4.1, C5.1, L3.2
- net FH2: now also L6.1, S3.1
- net FH4: now reaches C47.1, C48.1, C49.1, C50.1, C51.1, C52.1, L1.3, L2.3
- net FH4: now also S4.1
- net -12v PWM: no longer names the net of C20.1, C22.1, C24.1, C26.1, C28.2, C29.2, C30.2, C31.2, C32.2, C33.1, C35.1, C36.1, C37.1, C38.1, C39.1, C45.1, L2.2
- net -12v PWM: now also L6.4
- net Earth_Protective | GD renamed To GD
- net Line 220V renamed DC +12 or +5 V
- removed net Neutral: C1.2, C10.2, C12.2, C13.2, C14.2, C15.2, C16.2, C18.2, C2.2, C3.2, C4.2, C6.2, C7.2, C8.2, C9.2, L3.3, L3.4, L4.3, L4.4, L5.3, L5.4
- new net: C75.1, C78.1, C79.1, C82.1, C83.1, S1.4
- new net: C19.1, C76.1, C77.1, C80.1, C81.1, S1.2
- new net: C10.2, C12.2, C7.2, C8.2, C9.2, L3.3, L4.4
- new net: C84.1, C85.1, C86.1, C87.1, C88.1, S2.2
- new net: C89.1, C90.1, C91.1, C92.1, C93.1, S2.4
- new net: C13.2, C14.2, C15.2, C16.2, C18.2, L4.3, L5.4
- new net: C100.1, C101.1, C102.1, C103.1, C99.1, S3.4
- new net: C109.1, C110.1, C111.1, C112.1, C113.1, S4.4
- new net: C1.2, C2.2, C3.2, C4.2, C6.2, L3.4, L6.3
- new net: C94.1, C95.1, C96.1, C97.1, C98.1, S3.2
- new net: C104.1, C105.1, C106.1, C107.1, C108.1, S4.2
- new net DC "Ground": L5.3
- new net V-GND: C100.2, C101.2, C102.2, C103.2, C104.2, C105.2, C106.2, C107.2, C108.2, C109.2, C110.2, C111.2, C112.2, C113.2, C19.2, C75.2, C76.2, C77.2, C78.2, C79.2, C80.2, C81.2, C82.2, C83.2, C84.2, C85.2, C86.2, C87.2, C88.2, C89.2, C90.2, C91.2, C92.2, C93.2, C94.2, C95.2, C96.2, C97.2, C98.2, C99.2
Other:
- note added: "2024.12.03"
- note added: "Capacitor placement"
- note added: "Ground devices"
- note added: "OSH"
- note added: "Timers and relays (flip flop) from Grounding device but with capasitors instead resistors"
- note added: "workaround with DC power sources"
- note removed: "But this is not a solution of my problems criminals just continue to use and controll me from power sources with transformers or coils maybe I use transformerless in future"
- note removed: "Line"
- note removed: "PWM POWER SOURCE"
- note removed: "workaround with PWM power source"
- moved on the sheet: C1, C10, C11, C12, C13, C14, C15, C16, C17, C18, C2, C3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
